File: hardware/DC29-badge/DC29-badge.sch (KiCad schematic (older format))
At the start: 1 part, among them U1 STM32F746BGTx

Commit message: Change MCU component
We really do need to use the STM32F746NG part, not the BG one.
Parts:
- U1: value STM32F746BGTx -> STM32F746NGHx; footprint Package_QFP:LQFP-208_28x28mm_P0.5mm -> Package_BGA:TFBGA-216_13x13mm_Layout15x15_P0.8mm; symbol MCU_ST_STM32F7:STM32F746BGTx -> MCU_ST_STM32F7:STM32F746NGHx
Connections:
- wire segments 205 -> 200
